File: CQmax10/CQmax10.kicad_pcb (KiCad board)
At the start: 2 copper layers, 20 parts, among them CN1 Conn_02x25_Odd_Even, CN2 Conn_02x25_Odd_Even, J7 Conn_02x25_Odd_Even, J8 Conn_02x25_Odd_Even

Commit message: artwork
Parts:
- added J1: ~, kicad8-2:Pmod_socket, F.Cu at (156.2, 90.2)
- added J2: ~, kicad8-2:Pmod_socket, F.Cu at (172.1, 90.2)
- added J3: ~, kicad8-2:Pmod_socket, F.Cu at (188.0, 90.2)
- added J4: ~, kicad8-2:Pmod_socket, F.Cu at (203.9, 90.2)
- added J5: ~, kicad8-2:Pmod_socket, F.Cu at (219.8, 90.2)
- added J6: ~, kicad8-2:Pmod_socket, F.Cu at (235.7, 90.2)
- S1, S2, S3, S4: footprint samacsys:TVBP06B043CWB -> kicad8:TVBP06B043CWB

Commit message: schematics
Parts:
- moved J6 137.2 mm to (103.1, 54.9), turned to -90 degrees
- moved J5 114.4 mm to (118.9, 144.0), turned to 90 degrees
- moved J3 114.1 mm to (79.2, 55.7), turned to -90 degrees
- moved R1 104.2 mm to (153.8, 96.0), turned to 0 degrees
- moved R4 104.0 mm to (153.8, 79.5), turned to 0 degrees
- moved R2 103.5 mm to (153.8, 90.2), turned to 0 degrees
- moved R3 103.5 mm to (153.8, 84.6), turned to 0 degrees
- moved J1 99.7 mm to (72.2, 143.7), turned to 90 degrees
- moved D1 96.7 mm to (148.4, 96.0), turned to 180 degrees
- moved D4 96.4 mm to (148.4, 79.5), turned to 180 degrees
- moved D2 96.0 mm to (148.4, 90.2), turned to 180 degrees
- moved D3 95.9 mm to (148.4, 84.6), turned to 180 degrees
- moved J2 93.6 mm to (95.0, 143.2), turned to 90 degrees
- moved J4 87.2 mm to (124.2, 54.9), turned to -90 degrees
- moved S4 60.5 mm to (154.3, 115.2), turned to 180 degrees
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Connections:
- D1 pad 1: /IOPIN27 -> unconnected-(D1-K-Pad1)
- D2 pad 1: /IOPIN29 -> unconnected-(D2-K-Pad1)
- D3 pad 1: /IOPIN32 -> unconnected-(D3-K-Pad1)
- D4 pad 1: /IOPIN38 -> unconnected-(D4-K-Pad1)
- J1 pad 1: unconnected-(J1-Pin_1-Pad1) -> /IOPIN38
- J1 pad 10: unconnected-(J1-Pin_10-Pad10) -> /IOPIN47
- J1 pad 2: unconnected-(J1-Pin_2-Pad2) -> /IOPIN39
- J1 pad 3: unconnected-(J1-Pin_3-Pad3) -> /IOPIN41
- J1 pad 4: unconnected-(J1-Pin_4-Pad4) -> /IOPIN43
- J1 pad 7: unconnected-(J1-Pin_7-Pad7) -> /IOPIN44
- J1 pad 8: unconnected-(J1-Pin_8-Pad8) -> /IOPIN45
- J1 pad 9: unconnected-(J1-Pin_9-Pad9) -> /IOPIN46
- J2 pad 1: unconnected-(J2-Pin_1-Pad1) -> /IOPIN50
- J2 pad 10: unconnected-(J2-Pin_10-Pad10) -> /IOPIN60
- J2 pad 2: unconnected-(J2-Pin_2-Pad2) -> /IOPIN52
- J2 pad 3: unconnected-(J2-Pin_3-Pad3) -> /IOPIN55
- J2 pad 4: unconnected-(J2-Pin_4-Pad4) -> /IOPIN56
- J2 pad 7: unconnected-(J2-Pin_7-Pad7) -> /IOPIN57
- J2 pad 8: unconnected-(J2-Pin_8-Pad8) -> /IOPIN58
- J2 pad 9: unconnected-(J2-Pin_9-Pad9) -> /IOPIN59
- J3 pad 1: unconnected-(J3-Pin_1-Pad1) -> /IOPIN6
- J3 pad 10: unconnected-(J3-Pin_10-Pad10) -> /IOPIN14
- J3 pad 2: unconnected-(J3-Pin_2-Pad2) -> /IOPIN7
- J3 pad 3: unconnected-(J3-Pin_3-Pad3) -> /IOPIN8
- J3 pad 4: unconnected-(J3-Pin_4-Pad4) -> /IOPIN10
- J3 pad 7: unconnected-(J3-Pin_7-Pad7) -> /IOPIN11
- J3 pad 8: unconnected-(J3-Pin_8-Pad8) -> /IOPIN12
- J3 pad 9: unconnected-(J3-Pin_9-Pad9) -> /IOPIN13
- J4 pad 1: unconnected-(J4-Pin_1-Pad1) -> /IOPIN96
- J4 pad 10: unconnected-(J4-Pin_10-Pad10) -> /IOPIN106
- J4 pad 2: unconnected-(J4-Pin_2-Pad2) -> /IOPIN97
- J4 pad 3: unconnected-(J4-Pin_3-Pad3) -> /IOPIN98
- J4 pad 4: unconnected-(J4-Pin_4-Pad4) -> /IOPIN99
- J4 pad 7: unconnected-(J4-Pin_7-Pad7) -> /IOPIN100
- J4 pad 8: unconnected-(J4-Pin_8-Pad8) -> /IOPIN101
- J4 pad 9: unconnected-(J4-Pin_9-Pad9) -> /IOPIN105
- J5 pad 1: unconnected-(J5-Pin_1-Pad1) -> /IOPIN74
- J5 pad 10: unconnected-(J5-Pin_10-Pad10) -> /IOPIN81
- J5 pad 2: unconnected-(J5-Pin_2-Pad2) -> /IOPIN75
- J5 pad 3: unconnected-(J5-Pin_3-Pad3) -> /IOPIN76
- J5 pad 4: unconnected-(J5-Pin_4-Pad4) -> /IOPIN77
- J5 pad 7: unconnected-(J5-Pin_7-Pad7) -> /IOPIN78
- J5 pad 8: unconnected-(J5-Pin_8-Pad8) -> /IOPIN79
- J5 pad 9: unconnected-(J5-Pin_9-Pad9) -> /IOPIN80
- J6 pad 1: unconnected-(J6-Pin_1-Pad1) -> /IOPIN127
- J6 pad 10: unconnected-(J6-Pin_10-Pad10) -> /IOPIN141
- J6 pad 2: unconnected-(J6-Pin_2-Pad2) -> /IOPIN130
- J6 pad 3: unconnected-(J6-Pin_3-Pad3) -> /IOPIN131
- J6 pad 4: unconnected-(J6-Pin_4-Pad4) -> /IOPIN132
- J6 pad 7: unconnected-(J6-Pin_7-Pad7) -> /IOPIN134
- J6 pad 8: unconnected-(J6-Pin_8-Pad8) -> /IOPIN135
- J6 pad 9: unconnected-(J6-Pin_9-Pad9) -> /IOPIN140
- R5 pad 2: /IOPIN26 -> /IOPIN30
- R6 pad 2: /IOPIN28 -> /IOPIN48
- R7 pad 2: /IOPIN30 -> /IOPIN54
- R8 pad 2: /IOPIN33 -> /IOPIN62
- S1 pad 2: /IOPIN26 -> /IOPIN30
- S2 pad 2: /IOPIN28 -> /IOPIN48
- S3 pad 2: /IOPIN30 -> /IOPIN54
- S4 pad 2: /IOPIN33 -> /IOPIN62
Other:
- board outline added: 99.8 x 99.8 mm

Commit message: artwork
Parts:
- added REF**: MountingHole_3.2mm_M3, MountingHole:MountingHole_3.2mm_M3, F.Cu at (155.2, 59.9)
- added REF**: MountingHole_3.2mm_M3, MountingHole:MountingHole_3.2mm_M3, F.Cu at (65.3, 59.9)
- added REF**: MountingHole_3.2mm_M3, MountingHole:MountingHole_3.2mm_M3, F.Cu at (155.2, 149.6)
- added REF**: MountingHole_3.2mm_M3, MountingHole:MountingHole_3.2mm_M3, F.Cu at (65.3, 149.6)
- moved J4 17.1 mm to (135.4, 67.9)
- moved J3 16.0 mm to (89.6, 67.9)
- moved J6 16.0 mm to (112.5, 67.9)
- moved R7 14.3 mm to (146.8, 111.0)
- moved R8 14.3 mm to (146.8, 101.6)
- moved R6 14.2 mm to (146.8, 120.4), turned to 180 degrees
- moved R5 14.1 mm to (146.8, 129.5), turned to 180 degrees
- moved S1 9.00 mm to (152.3, 134.1)
- moved S2 8.98 mm to (152.4, 125.1)
- moved S3 8.98 mm to (152.3, 115.8)
- moved S4 8.98 mm to (152.3, 106.4)
- moved J7 6.98 mm to (69.3, 125.2)
- moved J8 6.88 mm to (69.3, 80.3)
- moved CN1 6.60 mm to (69.3, 132.1)
- moved J1 5.20 mm to (77.0, 141.7)
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Connections:
- D1 pad 1: unconnected-(D1-K-Pad1) -> /IOPIN123
- D2 pad 1: unconnected-(D2-K-Pad1) -> /IOPIN122
- D3 pad 1: unconnected-(D3-K-Pad1) -> /IOPIN120
- D4 pad 1: unconnected-(D4-K-Pad1) -> /IOPIN121
- J1 pad 1: /IOPIN38 -> /IOPIN46
- J1 pad 11: unconnected-(J1-Pin_11-Pad11) -> GND
- J1 pad 12: unconnected-(J1-Pin_12-Pad12) -> +3V3
- J1 pad 2: /IOPIN39 -> /IOPIN44
- J1 pad 4: /IOPIN43 -> /IOPIN38
- J1 pad 5: unconnected-(J1-Pin_5-Pad5) -> GND
- J1 pad 6: unconnected-(J1-Pin_6-Pad6) -> +3V3
- J1 pad 7: /IOPIN44 -> /IOPIN45
- J1 pad 8: /IOPIN45 -> /IOPIN43
- J1 pad 9: /IOPIN46 -> /IOPIN39
- J2 pad 1: /IOPIN50 -> /IOPIN59
- J2 pad 10: /IOPIN60 -> /IOPIN50
- J2 pad 11: unconnected-(J2-Pin_11-Pad11) -> GND
- J2 pad 12: unconnected-(J2-Pin_12-Pad12) -> +3V3
- J2 pad 2: /IOPIN52 -> /IOPIN57
- J2 pad 4: /IOPIN56 -> /IOPIN52
- J2 pad 5: unconnected-(J2-Pin_5-Pad5) -> GND
- J2 pad 6: unconnected-(J2-Pin_6-Pad6) -> +3V3
- J2 pad 7: /IOPIN57 -> /IOPIN60
- J2 pad 9: /IOPIN59 -> /IOPIN56
- J3 pad 1: /IOPIN6 -> /IOPIN13
- J3 pad 10: /IOPIN14 -> /IOPIN7
- J3 pad 11: unconnected-(J3-Pin_11-Pad11) -> GND
- J3 pad 12: unconnected-(J3-Pin_12-Pad12) -> +3V3
- J3 pad 2: /IOPIN7 -> /IOPIN11
- J3 pad 4: /IOPIN10 -> /IOPIN6
- J3 pad 5: unconnected-(J3-Pin_5-Pad5) -> GND
- J3 pad 6: unconnected-(J3-Pin_6-Pad6) -> +3V3
- J3 pad 7: /IOPIN11 -> /IOPIN14
- J3 pad 9: /IOPIN13 -> /IOPIN10
- J4 pad 1: /IOPIN96 -> /IOPIN98
- J4 pad 11: unconnected-(J4-Pin_11-Pad11) -> GND
- J4 pad 12: unconnected-(J4-Pin_12-Pad12) -> +3V3
- J4 pad 2: /IOPIN97 -> /IOPIN99
- J4 pad 3: /IOPIN98 -> /IOPIN96
- J4 pad 4: /IOPIN99 -> /IOPIN97
- J4 pad 5: unconnected-(J4-Pin_5-Pad5) -> GND
- J4 pad 6: unconnected-(J4-Pin_6-Pad6) -> +3V3
- J4 pad 7: /IOPIN100 -> /IOPIN101
- J4 pad 8: /IOPIN101 -> /IOPIN100
- J5 pad 1: /IOPIN74 -> /IOPIN80
- J5 pad 10: /IOPIN81 -> /IOPIN75
- J5 pad 11: unconnected-(J5-Pin_11-Pad11) -> GND
- J5 pad 12: unconnected-(J5-Pin_12-Pad12) -> +3V3
- J5 pad 2: /IOPIN75 -> /IOPIN79
- J5 pad 3: /IOPIN76 -> /IOPIN77
- J5 pad 4: /IOPIN77 -> /IOPIN76
- J5 pad 5: unconnected-(J5-Pin_5-Pad5) -> GND
- J5 pad 6: unconnected-(J5-Pin_6-Pad6) -> +3V3
- J5 pad 7: /IOPIN78 -> /IOPIN81
- J5 pad 8: /IOPIN79 -> /IOPIN78
- J5 pad 9: /IOPIN80 -> /IOPIN74
- J6 pad 1: /IOPIN127 -> /IOPIN134
- J6 pad 10: /IOPIN141 -> /IOPIN127
- J6 pad 11: unconnected-(J6-Pin_11-Pad11) -> GND
- J6 pad 12: unconnected-(J6-Pin_12-Pad12) -> +3V3
- J6 pad 2: /IOPIN130 -> /IOPIN135
- J6 pad 3: /IOPIN131 -> /IOPIN132
- J6 pad 4: /IOPIN132 -> /IOPIN130
- J6 pad 5: unconnected-(J6-Pin_5-Pad5) -> GND
- J6 pad 6: unconnected-(J6-Pin_6-Pad6) -> +3V3
- J6 pad 7: /IOPIN134 -> /IOPIN141
- J6 pad 8: /IOPIN135 -> /IOPIN140
- J6 pad 9: /IOPIN140 -> /IOPIN131
- R5 pad 2: /IOPIN30 -> /IOPIN62
- R6 pad 2: /IOPIN48 -> /IOPIN54
- R7 pad 2: /IOPIN54 -> /IOPIN48
- R8 pad 2: /IOPIN62 -> /IOPIN30
- S1 pad 2: /IOPIN30 -> /IOPIN62
- S2 pad 2: /IOPIN48 -> /IOPIN54
- S3 pad 2: /IOPIN54 -> /IOPIN48
- S4 pad 2: /IOPIN62 -> /IOPIN30
Routing:
- net +3V3: track 0.00 -> 348.7 mm, vias 0 -> 1
- net /IOPIN30: track 0.00 -> 87.0 mm
- net /IOPIN48: track 0.00 -> 70.9 mm, vias 0 -> 1
- net /IOPIN121: track 0.00 -> 64.4 mm
- net /IOPIN122: track 0.00 -> 64.0 mm, vias 0 -> 1
- net /IOPIN120: track 0.00 -> 63.8 mm, vias 0 -> 1
- net /IOPIN54: track 0.00 -> 63.7 mm
- net /IOPIN123: track 0.00 -> 61.0 mm
- net /IOPIN62: track 0.00 -> 56.2 mm
- net /IOPIN106: track 0.00 -> 43.7 mm
- net /IOPIN74: track 0.00 -> 42.5 mm
- net /IOPIN140: track 0.00 -> 42.0 mm
- net /IOPIN47: track 0.00 -> 41.7 mm
- net /IOPIN105: track 0.00 -> 38.6 mm
- net /IOPIN50: track 0.00 -> 38.6 mm
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- added copper zone on B.Cu, net GND
- added copper zone on F.Cu, net GND
Other:
- board text added: "#[120]"
- board text added: "#[121]"
- board text added: "#[122]"
- board text added: "#[123]"
- board text added: "#[130]"
- board text added: "#[48]"
- board text added: "#[54]"
- board text added: "#[62]"
- board text added: "10 | 8"
- board text added: "100 | 99"
- board text added: "101 | 98"
- board text added: "101|100"
- board text added: "105 | 96"
- board text added: "105|102"
- board text added: "106 | 97"
- board text added: "10| 8"
- board text added: "110|106"
- board text added: "112|111"
- board text added: "114|113"
- board text added: "119|118"
- board text added: "12 | 11"
- board text added: "121|120"
- board text added: "123|122"
- board text added: "126|124"
- board text added: "127 | 130"
- board text added: "12|11"
- board text added: "130|127"
- board text added: "131 | 132"
- board text added: "132|131"
- board text added: "135|134"
- board text added: "14 | 13"
- board text added: "140 | 135"
- board text added: "141 | 134"
- board text added: "141|140"
- board text added: "14|13"
- board text added: "1500 mil"
- board text added: "22.86mm"
- board text added: "27|26"
- board text added: "29|28"
- board text added: "32|30"
- board text added: "38 | 47"
- board text added: "38|33"
- board text added: "3V3"
- board text added: "3V3|3V3"
- board text added: "41 | 39"
- board text added: "41|39"
- board text added: "44 | 43"
- board text added: "44|43"
- board text added: "46 | 45"
- board text added: "46|45"
- board text added: "48|47"
- board text added: "52 | 50"
- board text added: "52|50"
- board text added: "55 | 56"
- board text added: "55|54"
- board text added: "57 | 58"
- board text added: "57|56"
- board text added: "59 | 60"
- board text added: "59|58"
- board text added: "61|60"
- board text added: "64|62"
- board text added: "66|65"
- board text added: "7 | 6"
- board text added: "70|69"
- board text added: "75|74"
- board text added: "76 | 75"
- board text added: "77 | 74"
- board text added: "77|76"
- board text added: "79 | 78"
- board text added: "79|78"
- board text added: "7|6"
- board text added: "80 | 81"
- board text added: "81|80"
- board text added: "91|90"
- board text added: "93|92"
- board text added: "97|96"
- board text added: "99|98"
- board text added: "Analog"
- board text added: "CQ-MAX10-A_Pmod Board Rev 0.1"
- board text added: "GND"
- board text added: "G|G"
- board text added: "Low Speed"

Commit message: adjust schematics
Routing:
- net GND: track 0.00 -> 37.6 mm, vias 0 -> 12
- net /IOPIN47: track 41.7 -> 41.1 mm

Commit message: add usb-c, 3v3regulater
Parts:
- added C1: 0.33u, Capacitor_SMD:C_0603_1608Metric_Pad1.08x0.95mm_HandSolder, F.Cu at (73.6, 99.6)
- added C2: 2.2u, Capacitor_SMD:C_0603_1608Metric_Pad1.08x0.95mm_HandSolder, F.Cu at (74.4, 110.7)
- added IC1: NJM2845DL1-33-TE1, samacsys:TO-252-3-L1, F.Cu at (81.6, 105.4)
- added J9: A295-CTRPB-1, samacsys:A295CTRPB1, F.Cu at (67.0, 103.1)
- S1, S2, S3, S4: footprint kicad8:TVBP06B043CWB -> samacsys:TVBP06B043CWB
Routing:
- net +3V3: track 348.7 -> 368.4 mm
- net Net-(IC1-VIN): track 0.00 -> 9.13 mm

Commit message: add 5v pad
Parts:
- added J10: Conn_01x01_Pin, Connector_PinHeader_2.54mm:PinHeader_1x01_P2.54mm_Vertical, F.Cu at (64.8, 70.6)
Routing:
- net Net-(IC1-VIN): track 9.13 -> 42.6 mm
Other:
- board text added: "5V"
